Commit message: docs: complete initial system documentation
- add public architecture and observation-mode documentation
 - document AMCL dependency, TF authority, topics, QoS, and runtime parameters
 - document particle clustering, GMM extraction, health, and evidence algorithms
- add HEROS 3W and SICK microScan3 Isaac Sim setup and validation guidance
 - add current system limitations and developer code-reference documentation
 - include RViz and Isaac Sim validation screenshots
 - update package-local Isaac and RViz instructions to match the validated fixture
 - document Fast DDS requirements for remote ROS 2 and RViz use
 - align scanner configuration and checked-in simulator assets with the validated setup
 - remove stale issue-oriented wording from public documentation
 - complete Phase B1 documentation milestone
Closes #47

File: src/hybrid_localization_isaac_sim/robot/heros_3w_isaac.urdf (robot description, URDF)
Before this commit: robot innok_heros_3w_isaac_stable, 6 links, 5 joints
Joints:
- joint base_scan_joint: origin xyz=0.95 0 0.28 rpy=0 0 0 -> xyz=0.95 0 0.10 rpy=0 0 0
